File: HDMI-MUX/HDMI-MUX.kicad_pcb (KiCad board)
At the start: 4 copper layers, 109.9 x 53.5 mm, 42 parts, among them J1 SERIAL, J2 UJC-HP-3-SMT-TR, J3 HDMI_IN, J4 HDMI_1, J5 HDMI_2, J6 HDMI_3, J7 HDMI_4, SW1 RST, SW2 SEL, SW3 FLASH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

Commit message: Update fab output
Connections:
- J3 pad 18: unconnected-(J3-Pad18) -> +5V
- J4 pad 18: unconnected-(J4-Pad18) -> +5V
- J5 pad 18: unconnected-(J5-Pad18) -> +5V
- J6 pad 18: unconnected-(J6-Pad18) -> +5V
- J7 pad 18: unconnected-(J7-Pad18) -> +5V
Routing:
- net +5V: track 0.00 -> 173.6 mm, vias 0 -> 5
- net Net-(R10-Pad1): track 78.6 -> 77.2 mm, vias 3 -> 2
Other:
- board text added: "HDMI-MUX v02 2022 Rion Gronberg"
- board text removed: "HDMI-MUX v01 2022 Rion Gronberg"
