File: HDMI-MUX/HDMI-MUX.kicad_sch (KiCad schematic)
At the start: 38 parts, among them J1 SERIAL, J2 UJC-HP-3-SMT-TR, J3 HDMI_IN, J4 HDMI_1, J5 HDMI_2, J6 HDMI_3, J7 HDMI_4, SW1 RST, SW2 SEL, SW3 FLASH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

Commit message: Update fab output
Connections:
- net +5V: now reaches J5.18
- net +5V: now also J3.18, J4.18, J6.18, J7.18
